Commit message: Added top plate without hole

File: urdf/husky.urdf.xacro (robot description, xacro)
@@ -57,5 +57,5 @@
   <xacro:arg name="cpr_urdf_extras" default="$(optenv CPR_URDF_EXTRAS empty.urdf)" />
   <!-- Included URDF/XACRO Files -->
-  <xacro:include filename="$(find husky_description)/urdf/decorations.urdf.xacro" />
+  <xacro:include filename="$(find fkie_husky_manipulation_simulation)/urdf/decorations.urdf.xacro" />
   <xacro:include filename="$(find husky_description)/urdf/wheel.urdf.xacro" />
   <xacro:include filename="$(find husky_description)/urdf/accessories/intel_realsense.urdf.xacro"/>

File: urdf/husky_panda.urdf.xacro (robot description, xacro)
@@ -7,5 +7,5 @@
   <xacro:panda_arm arm_id="panda" connected_to="panda_mount_link"/>
   <joint name="panda_mount_joint" type="fixed">
-    <origin xyz="0.389 0 0.23135" rpy="0 0 0"/>
+    <origin xyz="0.1 0.0 0.23135" rpy="0 0 0"/>
     <parent link="base_link"/>
     <child link="panda_mount_link" />
