Commit message: Added lasers and the respective plugins

File: urdf/decorations.urdf.xacro (robot description, xacro)
@@ -171,4 +171,58 @@
     <link name="top_plate_front_link"/>
     <link name="top_plate_rear_link"/>
+    <!-- laser front -->
+    <link name="laser_front">
+      <inertial>
+        <origin xyz="0 0 0" rpy="0 0 3.1415" />
+        <mass value="1" />
+        <inertia ixx="1.0" ixy="0.0" ixz="0.0" iyy="1.0" iyz="0.0" izz="1.0" />
+      </inertial>
+      <visual>
+        <origin xyz="0 0 -0.05" rpy="0 0 0" />
+        <geometry>
+          <mesh filename="package://fkie_husky_manipulation_simulation/meshes/accessories/hokuyo_ust10.stl" />
+        </geometry>
+        <material name="light_grey" />
+      </visual>
+      <collision>
+        <origin xyz="0 0 -0.05" rpy="0 0 0" />
+        <geometry>
+          <box size="0.1 0.1 0.1" />
+        </geometry>
+        <material name="light_grey" />
+      </collision>
+    </link>
+    <joint name="joint_base_link_laser_front" type="fixed">
+      <origin xyz="0.42 0.0 0.3" rpy="0 0 ${M_PI/2}" />
+      <parent link="base_link"/>
+      <child link="laser_front" />
+    </joint>
+    <!-- laser rear -->
+    <link name="laser_rear">
+      <inertial>
+        <origin xyz="0 0 0" rpy="0 0 0" />
+        <mass value="1" />
+        <inertia ixx="1.0" ixy="0.0" ixz="0.0" iyy="1.0" iyz="0.0" izz="1.0" />
+      </inertial>
+      <visual>
+        <origin xyz="0 0 -0.05" rpy="0 0 0" />
+        <geometry>
+          <mesh filename="package://fkie_husky_manipulation_simulation/meshes/accessories/hokuyo_ust10.stl" />
+        </geometry>
+        <material name="light_grey" />
+      </visual>
+      <collision>
+        <origin xyz="0 0 -0.05" rpy="0 0 0" />
+        <geometry>
+          <box size="0.1 0.1 0.1" />
+        </geometry>
+        <material name="light_grey" />
+      </collision>
+    </link>
+    <joint name="joint_base_link_laser_rear" type="fixed">
+      <origin xyz="-0.26 0.0 0.3" rpy="0 0 1.55" />
+      <parent link="base_link"/>
+      <child link="laser_rear" />
+    </joint>
   </xacro:macro>
 </robot>

File: urdf/husky.urdf.xacro (robot description, xacro)
@@ -23,5 +23,5 @@
 <robot name="husky"
   xmlns:xacro="http://ros.org/wiki/xacro">
-  <xacro:arg name="laser_enabled" default="$(optenv HUSKY_LMS1XX_ENABLED 0)" />
+  <!-- <xacro:arg name="laser_enabled" default="$(optenv HUSKY_LMS1XX_ENABLED 0)" />
   <xacro:arg name="laser_xyz" default="$(optenv HUSKY_LMS1XX_XYZ 0.2206 0.0 0.00635)" />
   <xacro:arg name="laser_rpy" default="$(optenv HUSKY_LMS1XX_RPY 0.0 0.0 0.0)" />
@@ -47,21 +47,21 @@
   <xacro:arg name="realsense_xyz" default="$(optenv HUSKY_REALSENSE_XYZ 0 0 0)" />
   <xacro:arg name="realsense_rpy" default="$(optenv HUSKY_REALSENSE_RPY 0 0 0)" />
-  <xacro:arg name="realsense_mount" default="$(optenv HUSKY_REALSENSE_MOUNT_FRAME sensor_arch_mount_link)" />
+  <xacro:arg name="realsense_mount" default="$(optenv HUSKY_REALSENSE_MOUNT_FRAME sensor_arch_mount_link)" /> -->
   <xacro:property name="husky_front_bumper_extend" value="$(optenv HUSKY_FRONT_BUMPER_EXTEND 0)" />
   <xacro:property name="husky_rear_bumper_extend" value="$(optenv HUSKY_REAR_BUMPER_EXTEND 0)" />
   <!-- Height of the sensor arch in mm.  Must be either 510 or 300 -->
-  <xacro:arg name="sensor_arch_height" default="$(optenv HUSKY_SENSOR_ARCH_HEIGHT 510)" />
-  <xacro:arg name="sensor_arch" default="$(optenv HUSKY_SENSOR_ARCH 0)" />
+  <!-- <xacro:arg name="sensor_arch_height" default="$(optenv HUSKY_SENSOR_ARCH_HEIGHT 510)" />
+  <xacro:arg name="sensor_arch" default="$(optenv HUSKY_SENSOR_ARCH 0)" /> -->
   <xacro:arg name="robot_namespace" default="$(optenv ROBOT_NAMESPACE /)" />
-  <xacro:arg name="urdf_extras" default="$(optenv HUSKY_URDF_EXTRAS empty.urdf)" />
-  <xacro:arg name="cpr_urdf_extras" default="$(optenv CPR_URDF_EXTRAS empty.urdf)" />
+  <!-- <xacro:arg name="urdf_extras" default="$(optenv HUSKY_URDF_EXTRAS empty.urdf)" />
+  <xacro:arg name="cpr_urdf_extras" default="$(optenv CPR_URDF_EXTRAS empty.urdf)" /> -->
   <!-- Included URDF/XACRO Files -->
   <xacro:include filename="$(find fkie_husky_manipulation_simulation)/urdf/decorations.urdf.xacro" />
   <xacro:include filename="$(find husky_description)/urdf/wheel.urdf.xacro" />
-  <xacro:include filename="$(find husky_description)/urdf/accessories/intel_realsense.urdf.xacro"/>
+  <!-- <xacro:include filename="$(find husky_description)/urdf/accessories/intel_realsense.urdf.xacro"/>
   <xacro:include filename="$(find husky_description)/urdf/accessories/sick_lms1xx_mount.urdf.xacro"/>
   <xacro:include filename="$(find husky_description)/urdf/accessories/sensor_arch.urdf.xacro"/>
   <xacro:include filename="$(find husky_description)/urdf/accessories/hokuyo_ust10.urdf.xacro"/>
-  <xacro:include filename="$(find husky_description)/urdf/accessories/vlp16_mount.urdf.xacro"/>
+  <xacro:include filename="$(find husky_description)/urdf/accessories/vlp16_mount.urdf.xacro"/> -->
   <xacro:property name="M_PI" value="3.14159"/>
   <!-- Base Size -->
@@ -144,5 +144,5 @@
     Add the primary and secondary lasers
   -->
-  <xacro:if value="$(arg laser_enabled)">
+  <!-- <xacro:if value="$(arg laser_enabled)">
     <xacro:sick_lms1xx_mount prefix="base"/>
     <xacro:sick_lms1xx frame="base_laser" topic="scan" robot_namespace="$(arg robot_namespace)"/>
@@ -161,9 +161,9 @@
       <child link="rear_laser_mount" />
     </joint>
-  </xacro:if>
+  </xacro:if> -->
   <!--
     Add front and back hokuyo UST10 Lidars
   -->
-  <xacro:if value="$(arg laser_ust10_front_enabled)">
+  <!-- <xacro:if value="$(arg laser_ust10_front_enabled)">
     <xacro:hokuyo_ust10_mount topic="$(arg laser_ust10_front_topic)" prefix="$(arg laser_ust10_front_prefix)" parent_link="$(arg laser_ust10_front_parent)">
       <origin xyz="$(arg laser_ust10_front_xyz)" rpy="$(arg laser_ust10_front_rpy)" />
@@ -174,10 +174,10 @@
       <origin xyz="$(arg laser_ust10_rear_xyz)" rpy="$(arg laser_ust10_rear_rpy)" />
     </xacro:hokuyo_ust10_mount>
-  </xacro:if>
+  </xacro:if> -->
   <!--
     Add the main sensor arch if the user has specifically enabled it, or if a sensor
     requires it for mounting
   -->
-  <xacro:property name="sensorbar_user_enabled" value="$(arg sensor_arch)" />
+  <!-- <xacro:property name="sensorbar_user_enabled" value="$(arg sensor_arch)" />
   <xacro:property name="sensorbar_needed_realsense" value="$(arg realsense_enabled)" />
   <xacro:property name="sensorbar_needed_lidar" value="$(arg laser_3d_enabled)" />
@@ -186,7 +186,7 @@
       <origin xyz="$(optenv HUSKY_SENSOR_ARCH_OFFSET 0 0 0)" rpy="$(optenv HUSKY_SENSOR_ARCH_RPY 0 0 0)"/>
     </xacro:sensor_arch>
-  </xacro:if>
+  </xacro:if> -->
   <!-- add the intel realsense to the sensor arch if needed -->
-  <xacro:if value="$(arg realsense_enabled)">
+  <!-- <xacro:if value="$(arg realsense_enabled)">
     <link name="realsense_mountpoint"/>
     <joint name="realsense_mountpoint_joint" type="fixed">
@@ -196,16 +196,16 @@
     </joint>
     <xacro:intel_realsense_mount prefix="camera" topic="realsense" parent_link="realsense_mountpoint"/>
-  </xacro:if>
+  </xacro:if> -->
   <!--
     Add the 3d laser to the sensor arch if needed
   -->
-  <xacro:if value="$(arg laser_3d_enabled)">
+  <!-- <xacro:if value="$(arg laser_3d_enabled)">
     <xacro:vlp16_mount prefix="" parent_link="sensor_arch_mount_link" topic="$(optenv HUSKY_LASER_3D_TOPIC points)">
       <origin xyz="$(arg laser_3d_xyz)" rpy="$(arg laser_3d_rpy)" />
     </xacro:vlp16_mount>
-  </xacro:if>
+  </xacro:if> -->
   <!-- Optional custom includes. -->
-  <xacro:include filename="$(arg urdf_extras)" />
+  <!-- <xacro:include filename="$(arg urdf_extras)" /> -->
   <!-- Optional for Clearpath internal softwares -->
-  <xacro:include filename="$(arg cpr_urdf_extras)" />
+  <!-- <xacro:include filename="$(arg cpr_urdf_extras)" /> -->
 </robot>

File: urdf/husky_panda.urdf.xacro (robot description, xacro)
@@ -24,4 +24,74 @@
       <robotParam>$(arg robot_namespace)/robot_description</robotParam>
     </plugin>
+  </gazebo>
+  <!-- Laser properties -->
+  <xacro:property name="laser_update_rate" value="10.0" />
+  <xacro:property name="laser_max_range" value="30.0" />
+  <xacro:property name="laser_samples" value="720" />
+  <!-- add lasers -->
+  <gazebo reference="laser_rear">
+    <turnGravityOff>false</turnGravityOff>
+    <sensor type="gpu_ray" name="laser_rear">
+      <update_rate>${laser_update_rate}</update_rate>
+      <ray>
+        <scan>
+          <horizontal>
+            <samples>${laser_samples}</samples>
+            <resolution>1</resolution>
+            <min_angle>${M_PI * 0.03}</min_angle>
+            <max_angle>${M_PI * 0.97}</max_angle>
+          </horizontal>
+        </scan>
+        <range>
+          <min>0.2</min>
+          <max>${laser_max_range}</max>
+          <resolution>0.01</resolution>
+        </range>
+        <noise>
+          <type>gaussian</type>
+          <mean>0.0</mean>
+          <stddev>0.01</stddev>
+        </noise>
+      </ray>
+      <plugin name="gazebo_ros_planar_lidar" filename="libgazebo_ros_gpu_laser.so">
+        <topicName>laser_rear</topicName>
+        <frameName>laser_rear</frameName>
+        <robotNamespace>$(arg robot_namespace)</robotNamespace>
+      </plugin>
+    </sensor>
+  </gazebo>
+  <gazebo reference="laser_front">
+    <turnGravityOff>false</turnGravityOff>
+    <sensor type="gpu_ray" name="laser_front">
+      <update_rate>${laser_update_rate}</update_rate>
+      <ray>
+        <scan>
+          <horizontal>
+            <samples>${laser_samples}</samples>
+            <resolution>1</resolution>
+            <min_angle>${M_PI}</min_angle>
+            <max_angle>${M_PI *2.0}</max_angle>
+          </horizontal>
+        </scan>
+        <range>
+          <min>0.2</min>
+          <max>${laser_max_range}</max>
+          <resolution>0.01</resolution>
+        </range>
+        <noise>
+          <type>gaussian</type>
+          <mean>0.0</mean>
+          <stddev>0.01</stddev>
+        </noise>
+      </ray>
+      <plugin name="gazebo_ros_planar_lidar" filename="libgazebo_ros_gpu_laser.so">
+        <topicName>laser_front</topicName>
+        <frameName>laser_front</frameName>
+        <robotNamespace>$(arg robot_namespace)</robotNamespace>
+      </plugin>
+    </sensor>
+  </gazebo>
+  <gazebo>
+    <enable_wind>false</enable_wind>
   </gazebo>
   <!-- <gazebo>

Commit message: Delete meshes

File: urdf/decorations.urdf.xacro (robot description, xacro)
@@ -54,5 +54,5 @@
         <origin xyz="0 0 0" rpy="0 0 0" />
         <geometry>
-          <mesh filename="package://fkie_husky_manipulation_simulation/meshes/top_chassis.dae" />
+          <mesh filename="package://husky_description/meshes/top_chassis.dae" />
         </geometry>
       </visual>
@@ -67,5 +67,5 @@
       <visual>
         <geometry>
-          <mesh filename="package://fkie_husky_manipulation_simulation/meshes/user_rail.dae" />
+          <mesh filename="package://husky_description/meshes/user_rail.dae" />
         </geometry>
       </visual>
@@ -82,5 +82,5 @@
         <visual>
           <geometry>
-            <mesh filename="package://fkie_husky_manipulation_simulation/meshes/bumper.dae" />
+            <mesh filename="package://husky_description/meshes/bumper.dae" />
           </geometry>
         </visual>
@@ -96,5 +96,5 @@
           <visual>
             <geometry>
-              <mesh filename="package://fkie_husky_manipulation_simulation/meshes/bumper_extension.dae" />
+              <mesh filename="package://husky_description/meshes/bumper_extension.dae" />
             </geometry>
           </visual>
@@ -112,5 +112,5 @@
         <visual>
           <geometry>
-            <mesh filename="package://fkie_husky_manipulation_simulation/meshes/bumper.dae" />
+            <mesh filename="package://husky_description/meshes/bumper.dae" />
           </geometry>
         </visual>
@@ -126,5 +126,5 @@
           <visual>
             <geometry>
-              <mesh filename="package://fkie_husky_manipulation_simulation/meshes/bumper_extension.dae" />
+              <mesh filename="package://husky_description/meshes/bumper_extension.dae" />
             </geometry>
           </visual>
@@ -141,5 +141,5 @@
         <origin xyz="0 0 0" rpy="0 0 0" />
         <geometry>
-          <mesh filename="package://fkie_husky_manipulation_simulation/meshes/top_plate.dae" />
+          <mesh filename="package://husky_description/meshes/top_plate.dae" />
         </geometry>
       </visual>
@@ -147,5 +147,5 @@
         <origin xyz="0 0 0" rpy="0 0 0"/>
         <geometry>
-          <mesh filename="package://fkie_husky_manipulation_simulation/meshes/top_plate.stl" />
+          <mesh filename="package://husky_description/meshes/top_plate.stl" />
         </geometry>
       </collision>
@@ -181,5 +181,5 @@
         <origin xyz="0 0 -0.05" rpy="0 0 0" />
         <geometry>
-          <mesh filename="package://fkie_husky_manipulation_simulation/meshes/accessories/hokuyo_ust10.stl" />
+          <mesh filename="package://husky_description/meshes/accessories/hokuyo_ust10.stl" />
         </geometry>
         <material name="light_grey" />
@@ -208,5 +208,5 @@
         <origin xyz="0 0 -0.05" rpy="0 0 0" />
         <geometry>
-          <mesh filename="package://fkie_husky_manipulation_simulation/meshes/accessories/hokuyo_ust10.stl" />
+          <mesh filename="package://husky_description/meshes/accessories/hokuyo_ust10.stl" />
         </geometry>
         <material name="light_grey" />
